File: Hardware/Amplificador_EEG/Amplificador_EEG_Master/Amplificador_EEG_Master.kicad_sch (KiCad schematic)
At the start: 20 parts, among them J1 VIN, J2 VOUT_opAmp, J3 VIN_opAmp, J4 IN+, J5 IN-, J6 REF, J7 Vout, J8 Mounting_Hole, U1 AD620

Commit message: Add files via upload
Parts:
- R2, R3, R4, R5: footprint EESTN5:R_0805 -> EESTN5:RES0.3
Changed lines of the file:
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@@
 			)
 		)
-		(property "Footprint" "EESTN5:R_0805"
+		(property "Footprint" "EESTN5:RES0.3"
 			(at 186.69 63.5 0)
 			(effects
@@
 			)
 		)
-		(property "Footprint" "EESTN5:R_0805"
+		(property "Footprint" "EESTN5:RES0.3"
 			(at 97.79 99.06 0)
 			(effects
@@
 			)
 		)
-		(property "Footprint" "EESTN5:R_0805"
+		(property "Footprint" "EESTN5:RES0.3"
 			(at 118.11 104.14 0)
 			(effects
@@
 			)
 		)
-		(property "Footprint" "EESTN5:R_0805"
+		(property "Footprint" "EESTN5:RES0.3"
 			(at 191.77 58.42 0)
 			(effects
