File: Hardware/MicroControlador_EEG/MicroControlador_EEG/MicroControlador_EEG.kicad_sch (KiCad schematic)
At the start: 42 parts, among them J1 VIN, J10 Servo2, J11 Servo3, J12 Servo4, J13 Servo5, J14 Servo6, J15 USB_B_Micro, J16 AUX_CH340, J17 Mounting_Hole, J18 Mounting_Hole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

Commit message: Add files via upload
Parts:
- C3: footprint EESTN5:CAP_ELEC_5x11mm -> EESTN5:CAP_ELEC_8x11.5mm
Connections:
- net +5V: now also J1.1 (Pin_1); no longer J1.2 (Pin_2)
- net GND: now also J1.2 (Pin_2); no longer J1.1 (Pin_1)
- net RXD: no longer U3.2 (TXD)
- net TXD: now also U3.2 (TXD)
Other:
- moved on the sheet: J1
Changed lines of the file:
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@@
 		)
 	)
-	(wire
-		(pts
-			(xy 46.99 130.81) (xy 46.99 133.35)
-		)
-		(stroke
-			(width 0)
-			(type default)
-		)
-	)
 	(bus
 		(pts
@@
 	(wire
 		(pts
+			(xy 43.18 133.35) (xy 40.64 133.35)
+		)
+		(stroke
+			(width 0)
+			(type default)
+		)
+	)
+	(wire
+		(pts
 			(xy 173.99 137.16) (xy 171.45 137.16)
 		)
@@
 		)
 	)
+	(wire
+		(pts
+			(xy 40.64 135.89) (xy 43.18 135.89)
+		)
+		(stroke
+			(width 0)
+			(type default)
+		)
+	)
 	(bus
 		(pts
@@
 	(wire
 		(pts
-			(xy 46.99 133.35) (xy 44.45 133.35)
-		)
-		(stroke
-			(width 0)
-			(type default)
-		)
-	)
-	(wire
-		(pts
 			(xy 96.52 129.54) (xy 86.36 129.54)
 		)
@@
 	(wire
 		(pts
-			(xy 46.99 138.43) (xy 46.99 135.89)
+			(xy 40.64 138.43) (xy 40.64 135.89)
 		)
 		(stroke
@@
 		)
 	)
-	(wire
-		(pts
-			(xy 46.99 135.89) (xy 44.45 135.89)
-		)
-		(stroke
-			(width 0)
-			(type default)
-		)
-	)
 	(bus
 		(pts
@@
 	(wire
 		(pts
+			(xy 40.64 133.35) (xy 40.64 130.81)
+		)
+		(stroke
+			(width 0)
+			(type default)
+		)
+	)
+	(wire
+		(pts
 			(xy 187.96 147.32) (xy 190.5 147.32)
 		)
@@
 		)
 	)
-	(label "RXD"
+	(label "TXD"
 		(at 257.81 45.72 0)
 		(fields_autoplaced yes)
@@
 			)
 		)
-		(property "Footprint" "EESTN5:CAP_ELEC_5x11mm"
+		(property "Footprint" "EESTN5:CAP_ELEC_8x11.5mm"
 			(at 87.3252 140.97 0)
 			(effects
@@
 	(symbol
 		(lib_id "Connector_Generic:Conn_01x02")
-		(at 39.37 135.89 180)
+		(at 48.26 133.35 0)
 		(unit 1)
 		(exclude_from_sim no)
@@
 		(dnp no)
 		(property "Reference" "J1"
-			(at 35.814 132.842 0)
+			(at 51.816 136.398 0)
 			(effects
 				(font
@@
 		)
 		(property "Value" "VIN"
-			(at 35.306 135.636 0)
+			(at 52.324 133.604 0)
 			(effects
 				(font
@@
 		)
 		(property "Footprint" "Connector_Molex:Molex_KK-254_AE-6410-02A_1x02_P2.54mm_Vertical"
-			(at 39.37 135.89 0)
+			(at 48.26 133.35 0)
 			(effects
 				(font
@@
 		)
 		(property "Datasheet" "~"
-			(at 39.37 135.89 0)
+			(at 48.26 133.35 0)
 			(effects
 				(font
@@
 		)
 		(property "Description" "Generic connector, single row, 01x02, script generated (kicad-library-utils/schlib/autogen/connector/)"
-			(at 39.37 135.89 0)
+			(at 48.26 133.35 0)
 			(effects
 				(font
@@
 	(symbol
 		(lib_id "power:GND")
-		(at 46.99 138.43 0)
+		(at 40.64 138.43 0)
 		(unit 1)
 		(exclude_from_sim no)
@@
 		(dnp no)
 		(property "Reference" "#PWR011"
-			(at 46.99 144.78 0)
+			(at 40.64 144.78 0)
 			(effects
 				(font
@@
 		)
 		(property "Value" "GND"
-			(at 46.99 142.494 0)
+			(at 40.64 142.494 0)
 			(effects
 				(font
@@
 		)
 		(property "Footprint" ""
-			(at 46.99 138.43 0)
+			(at 40.64 138.43 0)
 			(effects
 				(font
@@
 		)
 		(property "Datasheet" ""
-			(at 46.99 138.43 0)
+			(at 40.64 138.43 0)
 			(effects
 				(font
@@
 		)
 		(property "Description" "Power symbol creates a global label with name \"GND\" , ground"
-			(at 46.99 138.43 0)
+			(at 40.64 138.43 0)
 			(effects
 				(font
@@
 	(symbol
 		(lib_id "power:+5V")
-		(at 46.99 130.81 0)
+		(at 40.64 130.81 0)
 		(unit 1)
 		(exclude_from_sim no)
@@
 		(dnp no)
 		(property "Reference" "#PWR013"
-			(at 46.99 134.62 0)
+			(at 40.64 134.62 0)
 			(effects
 				(font
@@
 		)
 		(property "Value" "+5V"
-			(at 46.99 126.746 0)
+			(at 40.64 126.746 0)
 			(effects
 				(font
@@
 		)
 		(property "Footprint" ""
-			(at 46.99 130.81 0)
+			(at 40.64 130.81 0)
 			(effects
 				(font
@@
 		)
 		(property "Datasheet" ""
-			(at 46.99 130.81 0)
+			(at 40.64 130.81 0)
 			(effects
 				(font
@@
 		)
 		(property "Description" "Power symbol creates a global label with name \"+5V\""
-			(at 46.99 130.81 0)
+			(at 40.64 130.81 0)
 			(effects
 				(font
