File: Hardware/Fuente_EEG/Fuente_2_EEG/Fuente_2_EEG.kicad_pcb (KiCad board)
At the start: 2 copper layers, 56 x 29 mm, 24 parts, among them J1 Mounting_Hole, J3 Power_Jack, J4 Power_BAT, J5 Vout_opAmp, J6 Vout_uC, SW1 SW_DIP, U1 ICL7660

Commit message: Add files via upload
Parts:
- C1, C12, C4, C7, C8, C9: footprint EESTN5:CAP_ELEC_5x11mm -> EESTN5:CAP_ELEC_8x11.5mm
- U1: footprint Package_SO:SOIC-8_3.9x4.9mm_P1.27mm -> EESTN5:DIP-8; moved to F.Cu
- moved J1 25.4 mm to (144.7, 109.0)
- moved C2 17.2 mm to (176.6, 103.0), turned to 180 degrees
- moved C6 9.46 mm to (173.3, 110.0), turned to -90 degrees
- moved U1 9.38 mm to (164.7, 97.4), turned to 0 degrees
- moved C11 7.19 mm to (155.5, 92.4), turned to 0 degrees
- moved R1 6.35 mm to (158.4, 96.0)
- moved C10 5.70 mm to (142.5, 89.2)
- moved LM2 5.05 mm to (152.5, 89.6)
- moved G*** 4.32 mm to (178.1, 89.0)
- moved SW1 4.17 mm to (139.7, 103.2)
- moved C12 4.02 mm to (154.7, 96.8)
- moved C7 3.83 mm to (159.1, 104.6)
- moved J3 3.66 mm to (139.3, 93.8)
- moved J4 3.63 mm to (129.1, 107.0)
- moved C9 3.52 mm to (145.7, 96.8)
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Routing:
- net +5V: track 70.3 -> 86.7 mm
- net GND: track 0.00 -> 10.5 mm, vias 0 -> 2
- net VCC: track 30.3 -> 35.0 mm
- net +9V: track 22.8 -> 26.9 mm
- net -5V: track 18.6 -> 15.4 mm
- net Net-(U1-CAP+): track 14.6 -> 11.6 mm
- net Net-(U1-OSC): track 3.18 -> 5.27 mm
- net Net-(LED1-A): track 5.03 -> 3.78 mm
- net Net-(U1-CAP-): track 18.1 -> 16.9 mm
- net +7.5V: track 9.49 -> 8.64 mm
Other:
- board size 56 x 29 mm -> 56.8 x 30.4 mm

Commit message: Add files via upload
Parts:
- C4: footprint EESTN5:CAP_ELEC_8x11.5mm -> EESTN5:CAP_ELEC_5x11mm
- moved C2 1.58 mm to (175.0, 103.2), turned to 90 degrees
Routing:
- net GND: track 10.5 -> 0.00 mm, vias 2 -> 0
- net Net-(U1-OSC): track 5.27 -> 4.41 mm
Changed lines of the file:
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@@
 		)
 	)
-	(footprint "EESTN5:CAP_ELEC_8x11.5mm"
+	(footprint "EESTN5:CAP_ELEC_5x11mm"
 		(layer "F.Cu")
 		(at 167.6525 91.2 -90)
-		(descr "Capacitor, pol, cyl 8x11.5mm")
+		(descr "Capacitor, pol, cyl 5x11mm")
 		(property "Reference" "C4"
-			(at 0 -5.4 90)
-			(layer "F.SilkS")
-			(effects
-				(font
-					(size 0.8 0.8)
-					(thickness 0.15)
-					(bold yes)
-				)
-			)
-		)
-		(property "Value" "10u"
-			(at 0 -0.2 90)
-			(layer "F.SilkS")
-			(hide yes)
+			(at 0 -4.2 -90)
+			(layer "F.SilkS")
 			(effects
 				(font
@@
 			)
 		)
-		(property "Footprint" "EESTN5:CAP_ELEC_8x11.5mm"
-			(at 0 0 90)
+		(property "Value" "10u"
+			(at 0 4.2 -90)
+			(layer "F.SilkS")
+			(hide yes)
+			(effects
+				(font
+					(size 1.524 1.524)
+					(thickness 0.3048)
+				)
+			)
+		)
+		(property "Footprint" "EESTN5:CAP_ELEC_5x11mm"
+			(at 0 0 -90)
 			(layer "F.Fab")
 			(hide yes)
@@
 		)
 		(property "Datasheet" ""
-			(at 0 0 90)
+			(at 0 0 -90)
 			(layer "F.Fab")
 			(hide yes)
@@
 		)
 		(property "Description" "Unpolarized capacitor"
-			(at 0 0 90)
+			(at 0 0 -90)
 			(layer "F.Fab")
 			(hide yes)
@@
 		(attr through_hole)
 		(fp_line
-			(start 1.3 -2.2)
-			(end 2.5 -2.2)
+			(start 1 -1.1)
+			(end 2 -1.1)
 			(stroke
 				(width 0.3)
@@
 		)
 		(fp_line
-			(start -2.4 -3.5)
-			(end 2.4 -3.5)
+			(start -1.7 -2.2)
+			(end 1.7 -2.2)
 			(stroke
 				(width 0.3048)
@@
 		)
 		(fp_line
-			(start -1.8 -3.7)
-			(end 1.8 -3.7)
+			(start -1.3 -2.4)
+			(end 1.3 -2.4)
 			(stroke
 				(width 0.3048)
@@
 		)
 		(fp_line
-			(start -1.4 -3.9)
-			(end 1.4 -3.9)
-			(stroke
-				(width 0.3048)
-				(type solid)
-			)
-			(layer "F.SilkS")
-		)
-		(fp_line
-			(start -0.8 -4.1)
-			(end 0.9 -4.1)
+			(start -0.8 -2.6)
+			(end 0.8 -2.6)
 			(stroke
 				(width 0.3048)
@@
 		(fp_circle
 			(center 0 0)
-			(end -4.3 0)
+			(end 2.8 0)
 			(stroke
 				(width 0.3048)
@@
 		)
 		(pad "1" thru_hole rect
-			(at 0 1.75 270)
-			(size 1.8 1.8)
-			(drill 0.8)
+			(at 0 1 270)
+			(size 1.524 1.524)
+			(drill 0.65)
 			(layers "*.Cu" "*.Mask" "F.SilkS")
 			(remove_unused_layers no)
@@
 		)
 		(pad "2" thru_hole circle
-			(at 0 -1.75 270)
-			(size 1.8 1.8)
-			(drill 0.8)
+			(at 0 -1 270)
+			(size 1.524 1.524)
+			(drill 0.65)
 			(layers "*.Cu" "*.Mask" "F.SilkS")
 			(remove_unused_layers no)
@@
 			(pintype "passive")
 		)
-		(model "CAP_ELEC_8_11.5.wrl"
+		(model "CAP_ELEC_5_11.wrl"
 			(offset
 				(xyz 0 0 -0.2539999962)
@@
 	(footprint "EESTN5:C_0805"
 		(layer "B.Cu")
-		(at 176.6 103.025 180)
+		(at 175.025 103.1725 90)
 		(descr "SMT capacitor, 0805")
 		(property "Reference" "C2"
-			(at -2.9 0.025 0)
+			(at -2.9 0.025 90)
 			(layer "B.SilkS")
 			(effects
@@
 		)
 		(property "Value" "100n"
-			(at 0 -0.9906 360)
+			(at 0 -0.9906 90)
 			(layer "B.SilkS")
 			(hide yes)
@@
 		)
 		(property "Footprint" "EESTN5:C_0805"
-			(at 0 0 360)
+			(at 0 0 90)
 			(layer "B.Fab")
 			(hide yes)
@@
 		)
 		(property "Datasheet" ""
-			(at 0 0 360)
+			(at 0 0 90)
 			(layer "B.Fab")
 			(hide yes)
@@
 		)
 		(property "Description" "Unpolarized capacitor"
-			(at 0 0 360)
+			(at 0 0 90)
 			(layer "B.Fab")
 			(hide yes)
@@
 		(attr through_hole)
 		(fp_line
+			(start 2 -1)
+			(end 2 1)
+			(stroke
+				(width 0.127)
+				(type solid)
+			)
+			(layer "B.SilkS")
+		)
+		(fp_line
+			(start 1 -1)
+			(end 2 -1)
+			(stroke
+				(width 0.127)
+				(type solid)
+			)
+			(layer "B.SilkS")
+		)
+		(fp_line
+			(start -1 -1)
+			(end -2 -1)
+			(stroke
+				(width 0.15)
+				(type solid)
+			)
+			(layer "B.SilkS")
+		)
+		(fp_line
+			(start -2 -1)
+			(end -2 1)
+			(stroke
+				(width 0.15)
+				(type solid)
+			)
+			(layer "B.SilkS")
+		)
+		(fp_line
 			(start 2 1)
 			(end 1 1)
@@
 		)
 		(fp_line
-			(start 2 -1)
-			(end 2 1)
-			(stroke
-				(width 0.127)
-				(type solid)
-			)
-			(layer "B.SilkS")
-		)
-		(fp_line
-			(start 1 -1)
-			(end 2 -1)
-			(stroke
-				(width 0.127)
-				(type solid)
-			)
-			(layer "B.SilkS")
-		)
-		(fp_line
-			(start -1 -1)
-			(end -2 -1)
-			(stroke
-				(width 0.15)
-				(type solid)
-			)
-			(layer "B.SilkS")
-		)
-		(fp_line
 			(start -2 1)
 			(end -1 1)
@@
 			(layer "B.SilkS")
 		)
-		(fp_line
-			(start -2 -1)
-			(end -2 1)
-			(stroke
-				(width 0.15)
-				(type solid)
-			)
-			(layer "B.SilkS")
-		)
 		(pad "1" smd rect
-			(at 0.9525 0 180)
+			(at 0.9525 0 90)
 			(size 1.30048 1.4986)
 			(layers "B.Cu" "B.Paste" "B.Mask")
@@
 		)
 		(pad "2" smd rect
-			(at -0.9525 0 180)
+			(at -0.9525 0 90)
 			(size 1.30048 1.4986)
 			(layers "B.Cu" "B.Paste" "B.Mask")
@@
 	)
 	(segment
-		(start 173.6 94.775)
-		(end 173.625 94.75)
-		(width 0.75)
-		(layer "F.Cu")
-		(net 1)
-	)
-	(segment
-		(start 163.175 94.775)
-		(end 173.6 94.775)
-		(width 0.75)
-		(layer "F.Cu")
-		(net 1)
-	)
-	(via
-		(at 163.175 94.775)
-		(size 1.5)
-		(drill 1)
-		(layers "F.Cu" "B.Cu")
-		(free yes)
-		(net 1)
-	)
-	(via
-		(at 173.625 94.75)
-		(size 1.5)
-		(drill 1)
-		(layers "F.Cu" "B.Cu")
-		(net 1)
-	)
-	(segment
 		(start 137.1875 110.8525)
 		(end 141.2725 110.8525)
@@
 	)
 	(segment
-		(start 175.6475 103.025)
-		(end 175.6475 101.9975)
+		(start 173.94 99.94)
+		(end 172.2725 99.94)
 		(width 0.75)
 		(layer "B.Cu")
@@
 	)
 	(segment
-		(start 175.6475 101.9975)
-		(end 173.59 99.94)
+		(start 175.025 102.22)
+		(end 175.025 101.025)
 		(width 0.75)
 		(layer "B.Cu")
@@
 	)
 	(segment
-		(start 173.59 99.94)
-		(end 172.2725 99.94)
+		(start 175.025 101.025)
+		(end 173.94 99.94)
 		(width 0.75)
 		(layer "B.Cu")
@@
 	)
 	(segment
-		(start 169.4025 91.2)
-		(end 168.325 92.2775)
+		(start 168.6525 91.2)
+		(end 168.325 91.5275)
 		(width 0.75)
 		(layer "B.Cu")
@@
 	)
 	(segment
-		(start 168.325 92.2775)
+		(start 168.325 91.5275)
 		(end 168.325 103.225)
 		(width 0.75)
@@
 	)
 	(segment
+		(start 167.05 91.5975)
+		(end 167.05 99.1)
+		(width 0.75)
+		(layer "B.Cu")
+		(net 5)
+	)
+	(segment
+		(start 166.6525 91.2)
+		(end 167.05 91.5975)
+		(width 0.75)
+		(layer "B.Cu")
+		(net 5)
+	)
+	(segment
 		(start 167.05 99.1)
 		(end 166.21 99.94)
 		(width 0.75)
 		(layer "B.Cu")
-		(net 5)
-	)
-	(segment
-		(start 165.9025 91.2)
-		(end 167.05 92.3475)
-		(width 0.75)
-		(layer "B.Cu")
-		(net 5)
-	)
-	(segment
-		(start 167.05 92.3475)
-		(end 167.05 99.1)
-		(width 0.75)
-		(layer "B.Cu")
