File: Hardware/Fuente_EEG/Fuente_2_EEG/Fuente_2_EEG.kicad_pcb (KiCad board)
At the start: 2 copper layers, 56.8 x 50.2 mm, 25 parts, among them J1 BJ_V1, J2 BJ_V2, J3 TB_V1, J4 TB_V2, J5 VOUT, J6 Moutning Hole

Commit message: Fuente Update
Parts:
- removed LM_V2: ~, EESTN5:TO-220
- added U1: L7905, EESTN5:TO-220, F.Cu at (165.8, 75.0)
- moved J6 20.5 mm to (139.3, 92.2)
- moved R1 1.59 mm to (158.3, 99.2)
- moved R2 0.24 mm to (154.9, 86.1)
Connections:
- net /+V1_Regulated renamed Net-(LM_V1-VOUT)
- C1 pad 2: /+V2_Regulated -> GND
- C2 pad 2: /+V2_Regulated -> GND
- C3 pad 2: /+V2_Regulated -> GND
- C4 pad 2: /+V2_Regulated -> Net-(C4-Pad2)
- C5 pad 1: /+V2_SW_OUT -> GND
- C6 pad 1: /+V2_SW_OUT -> GND
- C7 pad 1: /+V2_Regulated -> GND
- C7 pad 2: /-V2 -> Net-(U1-VO)
- C8 pad 1: /+V2_Regulated -> Net-(C4-Pad2)
- C8 pad 2: /-V2 -> Net-(U1-VO)
- F2 pad 1: /-V2 -> Net-(U1-VO)
- J1 pad 2: /+V2_Regulated -> GND
- J1 pad 3: /+V2_Regulated -> GND
- J3 pad 2: /+V2_Regulated -> GND
- J5 pad 2: /+V2_Regulated -> GND
- LED1 pad 2: /+V2_Regulated -> GND
- LM_V1 pad 2: /+V2_Regulated -> GND
- R2 pad 1: /+V2_SW_OUT -> GND
- Switch_V2 pad 1: /+V2_SW_OUT -> GND
Routing:
- net /+V2_Regulated: track 143.9 -> 0.00 mm, vias 2 -> 0
- net /+V2_SW_OUT: track 37.4 -> 0.00 mm
- net /+V1_SW_IN: track 64.3 -> 42.5 mm
- net /+V1_SW_OUT: track 44.2 -> 64.7 mm, vias 2 -> 0
- net Net-(U1-VO): track 0.00 -> 19.8 mm
- net /-V2: track 88.0 -> 69.7 mm
- net Net-(C4-Pad2): track 0.00 -> 18.2 mm
- net GND: track 0.00 -> 5.94 mm
- net /+V2_SW_IN: track 41.6 -> 44.2 mm
- net Net-(LM_V1-VOUT): track 24.7 -> 25.9 mm
- net Net-(LED1-A): track 2.46 -> 3.34 mm
- added copper zone on B.Cu, net GND
