File: Hardware/Fuente_EEG/Fuente_2_EEG/Fuente_2_EEG.kicad_sch (KiCad schematic)
At the start: 23 parts, among them J1 Mounting_Hole, J3 Power_Jack, J4 Power_BAT, J5 Vout_opAmp, J6 Vout_uC, SW1 SW_DIP, U1 ICL7660

Commit message: Add files via upload
Parts:
- C1, C12, C4, C7, C8, C9: footprint EESTN5:CAP_ELEC_5x11mm -> EESTN5:CAP_ELEC_8x11.5mm
- U1: footprint Package_SO:SOIC-8_3.9x4.9mm_P1.27mm -> EESTN5:DIP-8
Changed lines of the file:
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@@
 			)
 		)
-		(property "Footprint" "EESTN5:CAP_ELEC_5x11mm"
+		(property "Footprint" "EESTN5:CAP_ELEC_8x11.5mm"
 			(at 207.9752 87.63 0)
 			(effects
@@
 			)
 		)
-		(property "Footprint" "EESTN5:CAP_ELEC_5x11mm"
+		(property "Footprint" "EESTN5:CAP_ELEC_8x11.5mm"
 			(at 152.0952 119.38 0)
 			(effects
@@
 			)
 		)
-		(property "Footprint" "EESTN5:CAP_ELEC_5x11mm"
+		(property "Footprint" "EESTN5:CAP_ELEC_8x11.5mm"
 			(at 225.7552 82.55 0)
 			(effects
@@
 			)
 		)
-		(property "Footprint" "EESTN5:CAP_ELEC_5x11mm"
+		(property "Footprint" "EESTN5:CAP_ELEC_8x11.5mm"
 			(at 152.0952 86.36 0)
 			(effects
@@
 			)
 		)
-		(property "Footprint" "EESTN5:CAP_ELEC_5x11mm"
+		(property "Footprint" "EESTN5:CAP_ELEC_8x11.5mm"
 			(at 107.6452 119.38 0)
 			(effects
@@
 			)
 		)
-		(property "Footprint" "EESTN5:CAP_ELEC_5x11mm"
+		(property "Footprint" "EESTN5:CAP_ELEC_8x11.5mm"
 			(at 107.6452 86.36 0)
 			(effects
@@
 			)
 		)
-		(property "Footprint" "Package_SO:SOIC-8_3.9x4.9mm_P1.27mm"
+		(property "Footprint" "EESTN5:DIP-8"
 			(at 196.85 83.82 0)
 			(effects

Commit message: Add files via upload
Parts:
- C4: footprint EESTN5:CAP_ELEC_8x11.5mm -> EESTN5:CAP_ELEC_5x11mm
Changed lines of the file:
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@@
 			)
 		)
-		(property "Footprint" "EESTN5:CAP_ELEC_8x11.5mm"
+		(property "Footprint" "EESTN5:CAP_ELEC_5x11mm"
 			(at 207.9752 87.63 0)
 			(effects
