File: Hardware/Fuente_EEG/Fuente_EEG/Fuente_EEG.kicad_sch (KiCad schematic)
At the start: 18 parts, among them J1 Vout_opAmp, J2 Power_BAT, J3 Power_Jack, J4 Mounting_Hole, J5 Mounting_Hole, J6 Vout_uC, U1 ICL7660

Commit message: Última Actualización de Hardware
Parts:
- removed J1: Vout_opAmp, Connector_Molex:Molex_KK-254_AE-6410-03A_1x03_P2.54mm_Vertical, symbol Connector:Conn_01x03_Pin
- removed J2: Power_BAT, EESTN5:BORNERA2_DUO, symbol Connector:Screw_Terminal_01x02
- removed J3: Power_Jack, Connector_BarrelJack:BarrelJack_Horizontal, symbol Connector:Barrel_Jack_Switch
- removed J4, J5: Mounting_Hole, EESTN5:hole_2mm, symbol Connector_Generic:Conn_01x01
- removed J6: Vout_uC, Connector_Molex:Molex_KK-254_AE-6410-02A_1x02_P2.54mm_Vertical, symbol Connector:Conn_01x02_Pin
- removed LED1: RED, EESTN5:led_3mm_red, symbol EESTN5:LED
- removed U1: ICL7660, Package_SO:SOIC-8_3.9x4.9mm_P1.27mm, symbol Regulator_SwitchedCapacitor:ICL7660
- added C5: 470u, EESTN5:CAP_ELEC_5x11mm, symbol Device:C
- added C6, C7: 100n, EESTN5:C_0805, symbol Device:C
- added C8: 100u, EESTN5:CAP_ELEC_5x11mm, symbol Device:C
- added D1: Green, EESTN5:led_3mm_green, symbol Device:LED
- added D2: Red, EESTN5:led_3mm_red, symbol Device:LED
- added J1: Barrel_Jack_V1, Connector_BarrelJack:BarrelJack_Horizontal, symbol Connector:Barrel_Jack_Switch
- added J2: Barrel_Jack_V2, Connector_BarrelJack:BarrelJack_Horizontal, symbol Connector:Barrel_Jack_Switch
- added J3: TB_V1, EESTN5:BORNERA2_DUO, symbol EESTN5:TB_1X2
- added J4: TB_V2, EESTN5:BORNERA2_DUO, symbol EESTN5:TB_1X2
- added J5: OUTPUT, Connector_Molex:Molex_KK-254_AE-6410-03A_1x03_P2.54mm_Vertical, symbol Connector_Generic:Conn_01x03
- added J6: OUTPUT_uC, Connector_Molex:Molex_KK-254_AE-6410-02A_1x02_P2.54mm_Vertical, symbol Connector_Generic:Conn_01x02
- added LM2: LM7805, MacroLib:TO-220-3_Vertical, symbol Logo_Romano:LM7805_Inverse
- added LM3: LM7805, MacroLib:TO-220-3_Vertical, symbol Logo_Romano:LM7805
- added R2: 100, EESTN5:R_0805, symbol EESTN5:R
- added R3, R4: 470, EESTN5:R_0805, symbol EESTN5:R
- added SW1, SW2: SW_SPDT, EESTN5:SW_SPDT_TH_Vertical, symbol EESTN5:SW_SPDT
- C12, C4: value 470u -> 100u
- C9: value 10u -> 470u
- LM1: value ~ -> LM7805; footprint EESTN5:SOT223-TAB2 -> MacroLib:TO-220-3_Vertical
- R1: value 330 -> 100
Connections:
- net Vcc is gone; now on net Vcc1: C1.1, C2.1, LM1.1 (VIN)
- net +5V: now also J5.3 (Pin_3), R3.1
- net -5V: now also C7.2, C8.2, D2.1 (K), J5.1 (Pin_1), LM2.3 (VOUT), R2.2; no longer C11.1, C12.1
- net GND: now also C9.2, R1.2, C5.1, C6.1, C7.1, C8.1, D1.1 (K), J1.2, J1.3, J2.1, J3.2, J4.1, J5.2 (Pin_2), J6.2 (Pin_2), LM2.2 (ADJ/GND), LM3.2 (ADJ/GND), R2.1, R4.1
- net Vcc1: now reaches C9.1
- net Vcc1: now also C10.1, LM3.1 (VIN), SW1.1 (A)
- new net: D1.2 (A), R3.2
- new net: D2.2 (A), R4.2
- new net -V2: J2.2, J2.3, J4.2, SW2.2 (B)
- new net POWER_uC: C11.1, C12.1, J6.1 (Pin_1), LM3.3 (VOUT)
- new net V1: J1.1, J3.1, SW1.2 (B)
- new net Vcc2: C5.2, C6.2, LM2.1 (VIN), SW2.1 (A)
- no-connect marks 1 -> 2
Other:
- note added: "EEG Power Source"
- note added: "LEDs"
- note added: "MicroController Power Source"
- note added: "POWER OUTPUT"
- note added: "Power Switches"
- note added: "V1 INPUT"
- note added: "V2 INPUT"
- note removed: "-5v Converter"
- note removed: "5v Converter"
- note removed: "LED Witness"
- note removed: "Power Supplies"
- note removed: "Vout opAmp"
- note removed: "Vout uC"
