File: Beta/Amplificador_EEG/Amplificador_EEG/Amplificador_EEG.kicad_sch (KiCad schematic)
At the start: 48 parts, among them J1 IN, J2 REF, J3 GND, J4 POWER, J5 OUTPUT, U1 LM358, U2 AD620, U3 LM358, U4 LM358, U5 LM358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

Commit message: Actualización Componentes PCBs
Parts:
- C2: footprint EESTN5:CAP_0.2 -> EESTN5:CAP_ELEC_5x11mm
- R2: footprint EESTN5:R_0805 -> EESTN5:R_1206
Changed lines of the file:
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@@
 			)
 		)
-		(property "Footprint" "EESTN5:R_0805"
+		(property "Footprint" "EESTN5:R_1206"
 			(at 193.04 40.64 0)
 			(effects
@@
 			)
 		)
-		(property "Footprint" "EESTN5:CAP_0.2"
+		(property "Footprint" "EESTN5:CAP_ELEC_5x11mm"
 			(at 112.7252 85.09 0)
 			(effects

Commit message: Actualización Amplificador
Parts:
- added J6: Mounting Hole, symbol Connector_Generic:Conn_01x01
- R2: footprint EESTN5:R_1206 -> EESTN5:RES0.3
- R26: footprint EESTN5:R_0805 -> EESTN5:RES0.3
Changed lines of the file:
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@@
 			)
 		)
-		(property "Footprint" "EESTN5:R_1206"
+		(property "Footprint" "EESTN5:RES0.3"
 			(at 193.04 40.64 0)
 			(effects
@@
 			)
 		)
-		(property "Footprint" "EESTN5:R_0805"
+		(property "Footprint" "EESTN5:RES0.3"
 			(at 168.91 132.08 0)
 			(effects
@@
 					(unit 1)
 				)
+			)
+		)
+	)
+	(symbol
+		(lib_id "Connector_Generic:Conn_01x01")
+		(at 33.02 161.29 180)
+		(unit 1)
+		(exclude_from_sim no)
+		(in_bom yes)
+		(on_board yes)
+		(dnp no)
+		(property "Reference" "J6"
+			(at 32.766 164.084 0)
+			(effects
+				(font
+					(size 1.27 1.27)
+				)
+			)
+		)
+		(property "Value" "Mounting Hole"
+			(at 38.354 166.37 0)
+			(effects
+				(font
+					(size 1.27 1.27)
+				)
+			)
+		)
+		(property "Footprint" ""
+			(at 33.02 161.29 0)
+			(effects
+				(font
+					(size 1.27 1.27)
+				)
+				(hide yes)
+			)
+		)
+		(property "Datasheet" "~"
+			(at 33.02 161.29 0)
+			(effects
+				(font
+					(size 1.27 1.27)
+				)
+				(hide yes)
+			)
+		)
+		(property "Description" "Generic connector, single row, 01x01, script generated (kicad-library-utils/schlib/autogen/connector/)"
+			(at 33.02 161.29 0)
+			(effects
+				(font
+					(size 1.27 1.27)
+				)
+				(hide yes)
+			)
+		)
+		(pin "1"
+		)
+		(instances
+			(project ""
+				(path "/141ddca8-9f7a-462f-b9ed-747d728ae61d"
+					(reference "J6")
+					(unit 1)
+				)
