File: Hardware/Amplificador_EEG/Amplificador_EEG/Amplificador_EEG.kicad_pcb (KiCad board)
At the start: 2 copper layers, 51.4 x 56.7 mm, 49 parts, among them J1 IN, J2 REF, J3 GND, J4 POWER, J5 OUTPUT, U1 LM358, U2 AD620, U3 LM358, U4 LM358, U5 LM358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

Commit message: Actualización Amplificador
Parts:
- added J6: Mounting Hole, EESTN5:hole_3mm, F.Cu at (153.3, 81.0)
- R2: footprint EESTN5:R_1206 -> EESTN5:RES0.3; moved to F.Cu
- R26: footprint EESTN5:R_0805 -> EESTN5:RES0.3; moved to F.Cu
- moved R26 7.99 mm to (161.5, 117.5), turned to 90 degrees
- moved R2 2.90 mm to (177.2, 79.3), turned to -90 degrees
- moved R27 2.52 mm to (156.8, 111.5), turned to 90 degrees
- moved R17 1.32 mm to (149.1, 111.0)
- moved R16 1.17 mm to (152.1, 110.1)
Routing:
- net +5V: track 167.1 -> 173.3 mm, vias 5 -> 3
- net /Offset_Ref: track 4.22 -> 7.98 mm
- net Net-(U4-IN1-): track 4.05 -> 5.02 mm
- net /NotchFilter_OUT: track 15.6 -> 14.8 mm
- net /AD620_Ref: track 6.32 -> 6.98 mm
- net GND: vias 7 -> 6
Other:
- board size 51.4 x 56.7 mm -> 52.1 x 59.1 mm

Commit message: Actualización de Dimensiones
Parts:
- moved C1 8.89 mm to (174.1, 98.8), turned to -90 degrees
- moved J5 5.74 mm to (173.7, 106.7)
- moved G*** 2.55 mm to (168.6, 113.7), turned to 0 degrees
- moved R2 1.36 mm to (175.8, 79.5)
- moved R3 1.32 mm to (175.5, 86.7), turned to -90 degrees
- moved R5 1.27 mm to (133.6, 78.8)
- moved D5 1.27 mm to (137.5, 78.8)
- moved J1 0.75 mm to (143.3, 97.8)
- moved J3 0.75 mm to (143.3, 109.8)
- moved J2 0.75 mm to (143.3, 85.7)
- moved J4 0.74 mm to (131.1, 72.8)
Routing:
- net /AD620_OUT: track 11.5 -> 21.4 mm
- net Net-(C1-Pad1): track 5.05 -> 12.6 mm
- net /OUTPUT: track 21.6 -> 15.6 mm
- net +5V: track 173.3 -> 170.1 mm
- net -5V: track 139.5 -> 138.1 mm
- net /AD620_Ref: track 6.98 -> 5.58 mm
- net GND: vias 6 -> 7
Other:
- board size 52.1 x 59.1 mm -> 48.4 x 59.1 mm
- board text removed: "Iván Romano Electroencefalógrafo E.E.S.T. N°5 {dblquote}2 de Abril{dblquote} Temperley 2025"

Commit message: Actual
Parts:
- added C7: 1n, EESTN5:C_0805, B.Cu at (142.6, 76.1)
- added C8: 1n, EESTN5:C_0805, B.Cu at (142.6, 71.5)
- added D6: C2v2, EESTN5:DO-41, F.Cu at (136.0, 63.7)
- added D7: 1N4007, EESTN5:DO-41, F.Cu at (150.2, 63.7)
- added D8: 1N4007, EESTN5:DO-41, F.Cu at (150.2, 67.5)
- added J7: DRL, Connector_BarrelJack:BarrelJack_Horizontal, F.Cu at (164.5, 76.3)
- added J8: Jail Hole, EESTN5:hole_2mm, F.Cu at (174.1, 66.0)
- added J9: Jail Hole, EESTN5:hole_2mm, F.Cu at (174.1, 76.8)
- added R10: 1M, EESTN5:RES0.3, B.Cu at (144.2, 84.0)
- added R15: 10k, EESTN5:R_0805, B.Cu at (137.1, 76.1)
- added R30: 330, EESTN5:R_0805, B.Cu at (131.9, 67.5)
- added R31: 100k, EESTN5:R_0805, B.Cu at (140.1, 76.1)
- added R32: 100k, EESTN5:R_0805, B.Cu at (140.1, 71.5)
- added R8: 1M, EESTN5:RES0.3, B.Cu at (147.4, 84.0)
- added U7: LM358, EESTN5:SSOP-8, B.Cu at (132.9, 74.1)
- C1: footprint EESTN5:CAP_ELEC_5x11mm -> EESTN5:CAP_ELEC_8x11.5mm
- J6: footprint EESTN5:hole_3mm -> EESTN5:hole_2mm
- moved J4 14.9 mm to (133.1, 87.6), turned to 90 degrees
- moved C1 13.2 mm to (173.1, 112.0)
- moved C4 12.0 mm to (158.1, 117.7)
- moved C6 12.0 mm to (172.1, 106.2)
- moved J3 12.0 mm to (143.6, 121.8)
- moved R12 12.0 mm to (164.6, 110.9)
- moved R14 12.0 mm to (161.3, 114.3)
- moved R2 12.0 mm to (176.1, 91.5)
- moved R9 12.0 mm to (169.1, 105.2)
- moved U2 12.0 mm to (165.4, 90.4)
- moved C2 12.0 mm to (166.7, 105.0)
- moved C3 12.0 mm to (164.4, 117.6)
- moved C5 12.0 mm to (158.1, 111.2)
- moved D1 12.0 mm to (167.9, 86.5)
- moved D2 12.0 mm to (167.9, 83.6)
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Routing:
- net /DRL_OUT: track 0.00 -> 41.7 mm
- net -5V: track 138.1 -> 171.7 mm, vias 3 -> 4
- net +5V: track 170.1 -> 202.6 mm
- net /IN+: track 16.3 -> 36.8 mm, vias 0 -> 2
- net /IN-: track 19.1 -> 38.6 mm
- net /DRL_IN: track 0.00 -> 17.6 mm
- net Net-(U7-Out2): track 0.00 -> 17.0 mm
- net Net-(U7-IN2-): track 0.00 -> 14.4 mm
- net /DRL_REF: track 0.00 -> 7.43 mm
- net Net-(U7-IN1-): track 0.00 -> 3.22 mm
- net Net-(C1-Pad1): track 12.6 -> 14.8 mm
- net Net-(R18-Pad2): track 14.0 -> 15.7 mm
- net /AD620_OUT: track 21.4 -> 22.8 mm
- net /INPUT: track 43.1 -> 41.8 mm
Other:
- board size 48.4 x 59.1 mm -> 49.6 x 78.1 mm
