File: Hardware/Amplificador_EEG/Amplificador_EEG/Amplificador_EEG.kicad_sch (KiCad schematic)
At the start: 49 parts, among them J1 IN, J2 REF, J3 GND, J4 POWER, J5 OUTPUT, J6 Mounting Hole, U1 LM358, U2 AD620, U3 LM358, U4 LM358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

Commit message: Actual
Parts:
- added C7, C8: 1n, EESTN5:C_0805, symbol EESTN5:C
- added D6: C2v2, EESTN5:DO-41, symbol Diode:ZPDxx
- added D7, D8: 1N4007, EESTN5:DO-41, symbol Device:D
- added J7: DRL, Connector_BarrelJack:BarrelJack_Horizontal, symbol Connector:Barrel_Jack_Switch
- added J8, J9: Jail Hole, EESTN5:hole_2mm, symbol Connector_Generic:Conn_01x01
- added R10, R8: 1M, EESTN5:RES0.3, symbol EESTN5:R
- added R15: 10k, EESTN5:R_0805, symbol EESTN5:R
- added R30: 330, EESTN5:R_0805, symbol EESTN5:R
- added R31, R32: 100k, EESTN5:R_0805, symbol EESTN5:R
- added U7: LM358, EESTN5:SSOP-8, symbol Logo_Romano:LM385
- C1: footprint EESTN5:CAP_ELEC_5x11mm -> EESTN5:CAP_ELEC_8x11.5mm
- J6: footprint (none) -> EESTN5:hole_2mm
Connections:
- net +5V: now also D8.1 (K), R30.1, U7.8 (+Vcc)
- net -5V: now also D7.2 (A), U7.4 (-Vcc)
- net GND: now also D6.1 (K), J7.2, J7.3
- net IN+: now also R8.1
- net IN-: now also R10.2
- new net: C7.1, C8.1, R31.1, R32.1, U7.7 (Out2)
- new net: C7.2, R15.2, R31.2, U7.6 (IN2-)
- new net: R15.1, U7.1 (Out1), U7.2 (IN1-)
- new net DRL_IN: R10.1, R8.2, U7.3 (IN1+)
- new net DRL_OUT: C8.2, D7.1 (K), D8.2 (A), J7.1, R32.2
- new net DRL_REF: D6.2 (A), R30.2, U7.5 (IN2+)
Other:
- note added: "DRL Output"
- note added: "DRL Voltage Reference"
- note added: "Diven Right Leg System"
- note added: "More info https://github.com/Romano047/Electroencefalograma-AD620.git"
- moved on the sheet: C1, C2, C3, C4, C5, C6, D1, D2, D3, D4, D5, J1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
